File: HifiAmp_TPA3255.kicad_sch (KiCad schematic)
At the start: 123 parts, among them J1 PVDD 48V IN — NEEDS_DATA, J2 RCA L SE, J3 RCA R SE, J301 SPK_L, J302 SPK_R, J4 VOLUME_REMOTE, Q301 NEEDS_DATA - P-MOS VDS>=100V, Q302 IXTK200N10L2, U1 LM5010ASD, U2 LM2940IMP-12/NOPB, U3 TLV1117-33IDCY, U4 OPA1612AIDR, U5 OPA1612AIDR, U6 TPA3255B, U7 TPS3802K33DCKR, U8 LM5069-2

Commit message: fix(protection): D301 must be bidirectional, and Q301 was over-constrained
Two corrections to the block just frozen.

Q301 is not held to VDS >= 100 V by the D301 clamp. During a clamp its
gate is held 15 V below its source by R305 and D302, so it conducts and
its VDS stays near zero. What the clamp does impose is 93.6 V on the
node, hence on U8 VIN, which is the 88 V ceiling analysis and stands.
Q301's real requirement is reverse blocking at 56 V plus margin.

Chasing that surfaced a real defect: a unidirectional TVS with its anode
on GND forward-conducts the moment the supply is connected backwards. It
shorts the source and blows F301, which defeats the whole point of Q301.
Switched to SMDJ58CA, electrically identical on the same datasheet row,
and bidirectional like the Device:D_TVS symbol already placed.

Co-Authored-By: Claude Opus 5 <noreply@anthropic.com>
Claude-Session: https://claude.ai/code/session_01NUH7zQZvRu9pq1jvTrNHEG
Parts:
- D301: value SMDJ58A -> SMDJ58CA; MPN SMDJ58A -> SMDJ58CA; Manufacturer (none) -> Littelfuse
- Q301: value NEEDS_DATA - P-MOS VDS>=100V -> NEEDS_DATA - P-MOS 100V 12A
Changed lines of the file:
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@@
 			)
 		)
-		(property "Value" "SMDJ58A"
+		(property "Value" "SMDJ58CA"
 			(at 279.4 322.58 0)
 			(effects
@@
 			)
 		)
-				(property "MPN" "SMDJ58A"
+				(property "MPN" "SMDJ58CA"
+			(at 279.4 320.04 0)
+			(effects (font (size 1.27 1.27)) (hide yes))
+		)
+				(property "Manufacturer" "Littelfuse"
 			(at 279.4 320.04 0)
 			(effects (font (size 1.27 1.27)) (hide yes))
@@
 			)
 		)
-		(property "Value" "NEEDS_DATA - P-MOS VDS>=100V"
+		(property "Value" "NEEDS_DATA - P-MOS 100V 12A"
 			(at 297.18 320.04 0)
 			(effects

Commit message: fix(schematic): Q301/Q302 pinout was wrong, and freeze Q301 (B2.9, B2.10)
Both transistors carried a *_GSD symbol, which declares pin 2 as Source.
Both parts actually chosen put the Drain on pin 2, the tab: IPP330P10NM
in TO-220-3 and IXTK200N10L2 in TO-264. Carried to the PCB that swaps
drain and source on both, leaving the body diode permanently forward
biased and neither the reverse protection nor the hot swap working. ERC
is blind to this: pin numbering means nothing to it.

Moved to Q_PMOS_GDS and Q_NMOS_GDS. The fix is geometrically neutral,
checked in Transistor_FET.kicad_sym before applying: both variants place
G at (-5.08, 0), D at (2.54, 5.08) and S at (2.54, -5.08), only the
numbers differ. The diff is three deleted lines; every (at ...) stays
context. The schematic holds only these two transistors.

Q301 = IPP330P10NM, Infineon OptiMOS P-channel TO-220-3. Datasheet has
no text layer, so it was read by rendering the pages. -100 V against the
56 V it must block reversed, 33 mOhm for 0.70 W at 4.6 A, VGS +/-20 V
against the 15 V D302 clamp. No SOA constraint: it is always either full
on or off, unlike Q302.

Recorded but not acted on: at 100 V a P-channel is roughly three times
worse than an N-channel, and an ideal diode controller would supply the
high side drive whose absence rejected the N-channel back in B2.3.

Co-Authored-By: Claude Opus 5 <noreply@anthropic.com>
Claude-Session: https://claude.ai/code/session_01NUH7zQZvRu9pq1jvTrNHEG
Parts:
- Q301: value NEEDS_DATA - P-MOS 100V 12A -> IPP330P10NM; symbol Transistor_FET:Q_PMOS_GSD -> Transistor_FET:Q_PMOS_GDS; MPN (none) -> IPP330P10NM; Manufacturer (none) -> Infineon
- Q302: symbol Transistor_FET:Q_NMOS_GSD -> Transistor_FET:Q_NMOS_GDS
Connections:
- net PVDD: now also Q302.3 (S); no longer Q302.2 (S)
- net PVDD_FUSED: now also Q301.2 (D); no longer Q301.3 (D)
- net PVDD_PROT: now also Q301.3 (S); no longer Q301.2 (S)
- net PVDD_SENSE: now also Q302.2 (D); no longer Q302.3 (D)
Changed lines of the file:
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@@
 	)
 	(symbol
-		(lib_id "Transistor_FET:Q_PMOS_GSD")
+		(lib_id "Transistor_FET:Q_PMOS_GDS")
 		(at 292.1 320.04 0)
 		(unit 1)
@@
 			)
 		)
-		(property "Value" "NEEDS_DATA - P-MOS 100V 12A"
+		(property "Value" "IPP330P10NM"
 			(at 297.18 320.04 0)
 			(effects
@@
 			)
 		)
+				(property "MPN" "IPP330P10NM"
+			(at 292.1 320.04 0)
+			(effects (font (size 1.27 1.27)) (hide yes))
+		)
+				(property "Manufacturer" "Infineon"
+			(at 292.1 320.04 0)
+			(effects (font (size 1.27 1.27)) (hide yes))
+		)
 		(instances
 			(project "HifiAmp_TPA3255"
@@
 	)
 	(symbol
-		(lib_id "Transistor_FET:Q_NMOS_GSD")
+		(lib_id "Transistor_FET:Q_NMOS_GDS")
 		(at 381 424.18 0)
 		(unit 1)

Commit message: feat(footprints): assign D301, Q301 and Q302, and redo the missing list
Diff is three lines: only the Footprint fields change.

Re-inventorying the schematic turned up more gaps than the plan recorded.
The LM5069 programming network and the gate clamp added in B2.3, B2.4 and
B2.6 were never assigned footprints at all: C325, C326, D302 and R305
through R310. Sixteen parts are still unassigned, not eight.

One of them is not routine: R306 is the 4 mOhm shunt, carrying 4.6 A
continuously and up to 15.4 A while the LM5069 limits. It needs a real
power shunt part and footprint, not a generic passive. Opened as D1.5.

Co-Authored-By: Claude Opus 5 <noreply@anthropic.com>
Claude-Session: https://claude.ai/code/session_01NUH7zQZvRu9pq1jvTrNHEG
Parts:
- D301: footprint (none) -> Diode_SMD:D_SMC
- Q301: footprint (none) -> Package_TO_SOT_THT:TO-220-3_Vertical
- Q302: footprint (none) -> Package_TO_SOT_THT:TO-264-3_Vertical
Changed lines of the file:
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@@
 			)
 		)
-		(property "Footprint" ""
+		(property "Footprint" "Diode_SMD:D_SMC"
 			(at 279.4 320.04 0)
 			(hide yes)
@@
 			)
 		)
-		(property "Footprint" ""
+		(property "Footprint" "Package_TO_SOT_THT:TO-220-3_Vertical"
 			(at 297.18 317.5 0)
 			(hide yes)
@@
 			)
 		)
-		(property "Footprint" ""
+		(property "Footprint" "Package_TO_SOT_THT:TO-264-3_Vertical"
 			(at 386.08 421.64 0)
 			(hide yes)

Commit message: feat(footprints): close D1.5, and correct an invented part number
The protection block passives are assigned: R305 through R310, C325, C326
and D302. C110 and C210 went with them. Four parts are left unassigned,
all of them D1.4 work: F301, J2, J3, J4. RV1 is not one of them, it is
deliberately off-board.

Three defects were found in the initial pass and fixed.

C325 carried MKS2C044701O00KSSD. That part does not exist: "O" is not a
WIMA tolerance code and no distributor lists it. It is now
MKS2B044701K00KSSD, 4.7 uF / 50 V / 10 %. The 63 V part that does exist
is a 20 % part and had to be rejected: it drops the startup margin to
1.25x, under the 1.30x this design holds itself to. Tolerance picks this
capacitor, not voltage.

C325 had also been moved from 3.9 to 4.7 uF with no documentation, while
the design notes still said 3.9 uF in ten places along with every number
derived from it. The value is right, since 3.9 uF is E24 and film series
do not carry it, but it stretches t_flt by 20.5 %. Recomputed throughout:
startup margin 1.41x instead of 1.30x, and Q302's SOA exposure goes from
318 to 422 ms, still far inside a curve guaranteed at 5 s.

C326 had no voltage rating at all, on PVDD_PROT, the most stressed node
in the schematic: it decouples U8's VIN and reaches 93.6 V while D301
clamps. Now 100nF/250V.

What sizes these passives is almost never power, it is voltage. R305 and
R307 stand at 78.6 V and 87.1 V during a clamp, so a 0603 rated 50 V
would be violated and they are 0805. Only R306 is power-sized.

C110 and C210 closed a NEEDS_DATA by calculation rather than by sourcing
a datasheet number: VMID is a 5 kOhm Thevenin source feeding four
non-inverting inputs, and its 9 nV/sqrt(Hz) of thermal noise is eight
times the OPA1612's own. That is what sets the capacitance, not a
reference design.

Verified independently of the MCP: footprints checked on disk, netlist
exported and reread to confirm VIN and SENSE sit either side of R306,
and ERC run before and after a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
Parts:
- C110, C210: value NEEDS_DATA -> 10uF/25V; footprint (none) -> Capacitor_SMD:C_0805_2012Metric
- C325: value 3.9uF -> 4.7uF; footprint (none) -> Capacitor_THT:C_Rect_L7.2mm_W7.2mm_P5.00mm_FKS2_FKP2_MKS2_MKP2; MPN (none) -> MKS2B044701K00KSSD
- C326: value 100nF -> 100nF/250V; footprint (none) -> Capacitor_SMD:C_1206_3216Metric
- D302: value 15V - NEEDS_DATA -> BZT52C15; footprint (none) -> Diode_SMD:D_SOD-123; MPN (none) -> BZT52C15
- R305, R307: footprint (none) -> Resistor_SMD:R_0805_2012Metric
- R306: footprint (none) -> Resistor_SMD:R_2512_6332Metric; MPN (none) -> WSL25124L000FEA
- R308, R309, R310: footprint (none) -> Resistor_SMD:R_0603_1608Metric
Changed lines of the file:
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@@
 			)
 		)
-		(property "Value" "NEEDS_DATA"
+		(property "Value" "10uF/25V"
 			(at 188.595 138.43 0)
 			(effects
@@
 			)
 		)
-		(property "Footprint" ""
+		(property "Footprint" "Capacitor_SMD:C_0805_2012Metric"
 			(at 188.9252 139.7 0)
 			(hide yes)
@@
 			)
 		)
-		(property "Value" "NEEDS_DATA"
+		(property "Value" "10uF/25V"
 			(at 188.595 227.33 0)
 			(effects
@@
 			)
 		)
-		(property "Footprint" ""
+		(property "Footprint" "Capacitor_SMD:C_0805_2012Metric"
 			(at 188.9252 228.6 0)
 			(hide yes)
@@
 			)
 		)
-		(property "Footprint" ""
+		(property "Footprint" "Resistor_SMD:R_0805_2012Metric"
 			(at 309.88 316.738 90)
 			(hide yes)
@@
 			)
 		)
-		(property "Value" "15V - NEEDS_DATA"
+		(property "Value" "BZT52C15"
 			(at 309.88 327.66 0)
 			(effects
@@
 			)
 		)
-		(property "Footprint" ""
+		(property "Footprint" "Diode_SMD:D_SOD-123"
 			(at 309.88 325.12 0)
 			(hide yes)
@@
 			)
 		)
+				(property "MPN" "BZT52C15"
+			(at 309.88 325.12 0)
+			(effects (font (size 1.27 1.27)) (hide yes))
+		)
 		(instances
 			(project "HifiAmp_TPA3255"
@@
 			)
 		)
-		(property "Footprint" ""
+		(property "Footprint" "Resistor_SMD:R_2512_6332Metric"
 			(at 355.6 405.638 90)
 			(hide yes)
@@
 			)
 		)
+				(property "MPN" "WSL25124L000FEA"
+			(at 355.6 403.86 0)
+			(effects (font (size 1.27 1.27)) (hide yes))
+		)
 		(instances
 			(project "HifiAmp_TPA3255"
@@
 			)
 		)
-		(property "Footprint" ""
+		(property "Footprint" "Resistor_SMD:R_0805_2012Metric"
 			(at 297.942 400.05 90)
 			(hide yes)
@@
 			)
 		)
-		(property "Footprint" ""
+		(property "Footprint" "Resistor_SMD:R_0603_1608Metric"
 			(at 297.942 410.21 90)
 			(hide yes)
@@
 			)
 		)
-		(property "Footprint" ""
+		(property "Footprint" "Resistor_SMD:R_0603_1608Metric"
 			(at 297.942 420.37 90)
 			(hide yes)
@@
 			)
 		)
-		(property "Footprint" ""
+		(property "Footprint" "Resistor_SMD:R_0603_1608Metric"
 			(at 345.44 451.358 90)
 			(hide yes)
@@
 			)
 		)
-		(property "Value" "3.9uF"
+		(property "Value" "4.7uF"
 			(at 330.835 452.12 0)
 			(effects
@@
 			)
 		)
-		(property "Footprint" ""
+		(property "Footprint" "Capacitor_THT:C_Rect_L7.2mm_W7.2mm_P5.00mm_FKS2_FKP2_MKS2_MKP2"
 			(at 331.1652 453.39 0)
 			(hide yes)
@@
 			)
 		)
+				(property "MPN" "MKS2B044701K00KSSD"
+			(at 330.2 449.58 0)
+			(effects (font (size 1.27 1.27)) (hide yes))
+		)
 		(instances
 			(project "HifiAmp_TPA3255"
@@
 			)
 		)
-		(property "Value" "100nF"
+		(property "Value" "100nF/250V"
 			(at 313.055 406.4 0)
 			(effects
@@
 			)
 		)
-		(property "Footprint" ""
+		(property "Footprint" "Capacitor_SMD:C_1206_3216Metric"
 			(at 313.3852 407.67 0)
 			(hide yes)

Commit message: feat(footprints): close D1.1 and D1.4, every part now has a footprint
The remaining four parts are assigned. J2, J3 and J4 needed a decision
rather than data, and the user picked JST XH at 2.5 mm. What decides it
is keying, not size: J4 carries six conductors including two grounds,
and a volume harness reconnected backwards after a teardown would put
the pot input on ground and its wiper on the input. That is a silent
fault, no damage, hard to find. A screw terminal cannot prevent it.

F301 needed a local footprint, since Fuse_Schurter_UMT250 targets
3 x 10.1 mm against 5.3 x 16 mm here. Web search returned the numbers
from Schurter's pad drawing but could not attribute them to any
dimension, the leader labels not being extractable. Reading the PDF's
vector geometry directly settled it: the two pads, their edges and the
dimension arrows.

That reading also showed the drawing is not to scale. Measured, the
pad-to-gap ratio is 0.312 while the labels say 0.375, so the labels
govern. Three independent cross-checks confirm they are consistent: the
10.00 mm inner gap brackets the 9.80 mm of bare ceramic, each pad covers
2.70 of the 2.80 mm terminal, and overhangs 1.05 mm for the fillet.
Taking the drawing to scale would have cut terminal coverage by 20 %.

RV1 is not a gap. It is deliberately off-board, so only the PWR_FLAG
symbols are left without a footprint, and they need none.

Copper, paste, mask and courtyard on the new footprint are exact. Its
silkscreen and fab layers are not: the MCP's create_footprint imposes
its own graphics and no tool can edit them afterwards, so the fuse
carries a pin-1 marker although it is not polarized, with its circle
landing outside the courtyard. Left as generated rather than editing the
library by hand, which the project's rules forbid. Tracked in D1.8,
together with CF_Film_Box, whose courtyard is 2.6 mm for a 3.5 mm body
and would let DRC pass a part placed too close to C321-C324.

Verified independently of the MCP throughout: footp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
Parts:
- F301: footprint (none) -> HifiAmp_TPA3255_Local:Fuse_Schurter_UMT-H_5.3x16mm
- J2, J3: footprint (none) -> Connector_JST:JST_XH_B2B-XH-A_1x02_P2.50mm_Vertical
- J4: footprint (none) -> Connector_JST:JST_XH_B6B-XH-A_1x06_P2.50mm_Vertical
Changed lines of the file:
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@@
 			)
 		)
-		(property "Footprint" ""
+		(property "Footprint" "Connector_JST:JST_XH_B2B-XH-A_1x02_P2.50mm_Vertical"
 			(at 30.48 170.18 0)
 			(hide yes)
@@
 			)
 		)
-		(property "Footprint" ""
+		(property "Footprint" "Connector_JST:JST_XH_B2B-XH-A_1x02_P2.50mm_Vertical"
 			(at 30.48 259.08 0)
 			(hide yes)
@@
 			)
 		)
-		(property "Footprint" ""
+		(property "Footprint" "HifiAmp_TPA3255_Local:Fuse_Schurter_UMT-H_5.3x16mm"
 			(at 264.922 320.04 90)
 			(hide yes)
@@
 			)
 		)
-		(property "Footprint" ""
+		(property "Footprint" "Connector_JST:JST_XH_B6B-XH-A_1x06_P2.50mm_Vertical"
 			(at 15.24 209.55 0)
 			(hide yes)
