File: HifiAmp_TPA3255.kicad_pcb (KiCad board)
At the start: 4 copper layers, 200 x 150 mm, 124 parts, among them J1 PVDD 48V IN — NEEDS_DATA, J2 RCA L SE, J3 RCA R SE, J301 SPK_L, J302 SPK_R, J4 VOLUME_REMOTE, Q301 IPP330P10NM, Q302 IXTK200N10L2, U1 LM5010ASD, U2 LM2940IMP-12/NOPB, U3 TLV1117-33IDCY, U4 OPA1612AIDR, U5 OPA1612AIDR, U6 TPA3255B, U7 TPS3802K33DCKR, U8 LM5069-2

Commit message: feat(f1.1): turn C310 the right way round and route PVDD
C310 rotates 90 to -90 without moving, and its pads trade nets: PVDD now
sits at 176.825 facing U6 pins 36-38, which takes the decoupling loop from
9.04 mm with a crossing down to 7.71 mm without — the same figure C311
already had. PVDD then routes on F.Cu in four segments, no via, 0.8 mm
inside the channel BST_B borders and 1.1 mm past x=279.9 where the
bootstrap no longer runs, wide enough to cover all three pads at once.

The audit the user asked for came back reassuring. Crossing position with
orientation over the eight mirrored pairs, only three are discriminating —
the ones whose rotation is neither 0 nor 180, the only angles where a
mirror is visible at all. C306/C309 and C307/C308 are correct, so C310 was
the board's only orientation defect; everything else sits at 0 or 180,
where -theta equals theta and no such defect can exist.

Clearance belongs to the net class, and PWR_48V wants 0.5 mm where
GATE_DRIVE wants 0.25. The corridor in the brief had been computed with the
neighbour's figure, and a first 1.4 mm run answered with three clearance
violations at 0.2875 — which is what established the real bound.

GND stays unrouted here on purpose. BST_B crosses the upper GND corridor at
about x=279.72, BST_C the lower one by symmetry, so no local ground link
reaches C310 or C311 without a via. The returns go to the F1.4 plane, which
is the ordinary answer on four layers and keeps both sides symmetric.

Unconnected items drop 250 to 244, six and not two: each link resolves
three ratsnest lines, the three U6 pads plus the capacitor.

Co-Authored-By: Claude Opus 5 <noreply@anthropic.com>
Claude-Session: https://claude.ai/code/session_019BebeZkXR3UXsLfHa8ZWyd
Parts:
- turned C310 to -90 degrees
Routing:
- net /PVDD: track 0.00 -> 7.58 mm
Changed lines of the file:
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@@
 	(footprint "Capacitor_SMD:C_1210_3225Metric"
 		(layer "F.Cu")
-		(at 277.5 178.3 90)
+		(at 277.5 178.3 -90)
 		(descr "Capacitor SMD 1210 (3225 Metric), square (rectangular) end terminal, IPC-7351 nominal, (Body size source: IPC-SM-782 page 76, https://www.pcb-3d.com/wordpress/wp-content/uploads/ipc-sm-782a_amendment_1_and_2.pdf)")
 		(tags "capacitor")
 		(property "Reference" "C310"
-			(at 0 -2.3 90)
+			(at 0 -2.3 -90)
 			(layer "F.SilkS")
 			(effects
@@
 		)
 		(property "Value" "1uF/100V"
-			(at 0 2.3 90)
+			(at 0 2.3 -90)
 			(layer "F.Fab")
 			(effects
@@
 		)
 		(property "Datasheet" ""
-			(at 0 0 90)
+			(at 0 0 -90)
 			(layer "F.Fab")
 			(hide yes)
@@
 		)
 		(property "Description" ""
-			(at 0 0 90)
+			(at 0 0 -90)
 			(layer "F.Fab")
 			(hide yes)
@@
 		)
 		(property "KiLib_Generator" "SMD_2terminal_chip_molded"
-			(at 0 0 90)
+			(at 0 0 -90)
 			(layer "F.SilkS")
 			(hide yes)
@@
 		(sheetname "/")
 		(sheetfile "HifiAmp_TPA3255.kicad_sch")
-		(units
-			(unit
-				(name "A")
-				(pins "1" "2")
-			)
-		)
 		(attr smd)
 		(duplicate_pad_numbers_are_jumpers no)
 		(fp_line
-			(start -0.711252 -1.36)
-			(end 0.711252 -1.36)
+			(start -0.711252 1.36)
+			(end 0.711252 1.36)
 			(stroke
 				(width 0.12)
@@
 		)
 		(fp_line
-			(start -0.711252 1.36)
-			(end 0.711252 1.36)
+			(start -0.711252 -1.36)
+			(end 0.711252 -1.36)
 			(stroke
 				(width 0.12)
@@
 		)
 		(fp_text user "${REFERENCE}"
-			(at 0 0 90)
+			(at 0 0 -90)
 			(layer "F.Fab")
 			(effects
@@
 		)
 		(pad "1" smd roundrect
-			(at -1.475 0 90)
+			(at -1.475 0 270)
 			(size 1.15 2.7)
 			(layers "F.Cu" "F.Mask" "F.Paste")
@@
 		)
 		(pad "2" smd roundrect
-			(at 1.475 0 90)
+			(at 1.475 0 270)
 			(size 1.15 2.7)
 			(layers "F.Cu" "F.Mask" "F.Paste")
@@
 	)
 	(segment
+		(start 279.9 177.2225)
+		(end 281.2875 177.2225)
+		(width 1.1)
+		(layer "F.Cu")
+		(net "/PVDD")
+	)
+	(segment
+		(start 279.9 172.7775)
+		(end 281.2875 172.7775)
+		(width 1.1)
+		(layer "F.Cu")
+		(net "/PVDD")
+	)
+	(segment
+		(start 277.5 177.2225)
+		(end 279.9 177.2225)
+		(width 0.8)
+		(layer "F.Cu")
+		(net "/PVDD")
+	)
+	(segment
+		(start 277.5 172.7775)
+		(end 279.9 172.7775)
+		(width 0.8)
+		(layer "F.Cu")
+		(net "/PVDD")
+	)
+	(segment
